Commit message: Refactor project structure and imporve bringup package

File: icart_mini_description/urdf/icart.urdf (robot description, URDF)
Before this commit: robot icart_mini, 4 links, 3 joints
Joints:
- removed joint left_wheel_hinge
- removed joint right_wheel_hinge
- added joint left_wheel_joint: type continuous, parent base_link, child left_wheel, origin xyz=0 0.1 0.075 rpy=-1.5707963267948966 0 0, axis 0 0 1
- added joint right_wheel_joint: type continuous, parent base_link, child right_wheel, origin xyz=0 -0.1 0.075 rpy=-1.5707963267948966 0 0, axis 0 0 1

File: icart_mini_description/urdf/icart_mini.xacro (robot description, xacro)
@@ -46,5 +46,5 @@
   </link>
   <!-- Left Wheel -->
-  <joint type="continuous" name="left_wheel_hinge">
+  <joint type="continuous" name="left_wheel_joint">
     <axis xyz="0 0 1"/>
     <parent link="base_link"/>
@@ -63,5 +63,5 @@
   </link>
   <!-- Right Wheel -->
-  <joint type="continuous" name="right_wheel_hinge">
+  <joint type="continuous" name="right_wheel_joint">
     <axis xyz="0 0 1"/>
     <parent link="base_link"/>
