Commit message: Add scan joint at xacro

File: icart_mini_description/urdf/icart_mini.xacro (robot description, xacro)
@@ -79,3 +79,21 @@
     </visual>
   </link>
+  <!-- LiDAR -->
+  <joint name="scan_joint" type="fixed">
+    <axis xyz="0 1 0"/>
+    <origin xyz="0 0 0.2" rpy="0 0 0 "/>
+    <parent link="base_link"/>
+    <child link="base_scan"/>
+  </joint>
+  <link name="base_scan">
+    <visual>
+      <origin xyz="0 0 0" rpy="0 0 0 "/>
+      <geometry>
+        <box size="0.1 0.1 0.1"/>
+      </geometry>
+      <material name="red">
+        <color rgba="1 0 0 1"/>
+      </material>
+    </visual>
+  </link>
 </robot>

Commit message: Add urg node frame

File: icart_mini_description/urdf/icart_mini.xacro (robot description, xacro)
@@ -20,8 +20,8 @@
       <origin xyz="0 0 ${base_height}" rpy="0 0 0"/>
       <geometry>
-        <box size="0.35 0.18 0.4"/>
+        <box size="0.4 0.18 0.4"/>
       </geometry>
       <material name="white">
-        <color rgba="1.0 1.0 1.0 1.0"/>
+        <color rgba="1.0 1.0 1.0 0.5"/>
       </material>
     </visual>
@@ -41,5 +41,5 @@
       </geometry>
       <material name="white">
-        <color rgba="1.0 1.0 1.0 1.0"/>
+        <color rgba="1.0 1.0 1.0 0.5"/>
       </material>
     </visual>
@@ -58,5 +58,5 @@
       </geometry>
       <material name="gray">
-        <color rgba="0.2 0.2 0.2 1"/>
+        <color rgba="0.2 0.2 0.2 1.0"/>
       </material>
     </visual>
@@ -82,9 +82,9 @@
   <joint name="scan_joint" type="fixed">
     <axis xyz="0 1 0"/>
-    <origin xyz="0 0 0.2" rpy="0 0 0 "/>
+    <origin xyz="0.15 0 0.18" rpy="0 0 0 "/>
     <parent link="base_link"/>
-    <child link="base_scan"/>
+    <child link="laser"/>
   </joint>
-  <link name="base_scan">
+  <link name="laser">
     <visual>
       <origin xyz="0 0 0" rpy="0 0 0 "/>
@@ -93,5 +93,5 @@
       </geometry>
       <material name="red">
-        <color rgba="1 0 0 1"/>
+        <color rgba="1 0 0 0.5"/>
       </material>
     </visual>
