Commit message: FollowMe シミュレーションのジョイスティック操作と起動手順を追加
- Gazebo/RViz/脚モデル/追従ノードをまとめて起動する launch を追加
- Logitech F710 で icart 操作から人物操作へ切り替える teleop を追加
- 実機 README の Follow me ボタン割当に合わせて追従開始/停止を整理
- Docker からジョイスティックを認識できるよう /dev/input をマウント
- Gazebo 上で /cmd_vel により icart が移動するよう車輪接触設定を調整

File: icart_mini_description/urdf/icart_mini_gazebo.xacro (robot description, xacro)
@@ -18,5 +18,5 @@
   <xacro:property name="base_collision_center_z" value="0.08"/>
   <xacro:property name="base_height" value="0.25"/>
-  <xacro:property name="wheel_height" value="0.075"/>
+  <xacro:property name="wheel_height" value="${wheel_radius}"/>
   <xacro:property name="laser_x" value="0.15"/>
   <xacro:property name="laser_y" value="0.0"/>
@@ -169,7 +169,11 @@
   <gazebo reference="left_wheel">
     <material>Gazebo/DarkGrey</material>
+    <mu1>1.0</mu1>
+    <mu2>1.0</mu2>
   </gazebo>
   <gazebo reference="right_wheel">
     <material>Gazebo/DarkGrey</material>
+    <mu1>1.0</mu1>
+    <mu2>1.0</mu2>
   </gazebo>
   <gazebo reference="laser">
